File: MCU.kicad_sch (KiCad schematic)
At the start: 2 parts, among them SW1 SW_DIP_x01, U1 Pico

Commit message: ordered pcbs
Changed lines of the file:
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@@
     (effects (font (size 1.27 1.27)) (justify left bottom))
-  )
-  (label "Please check SPI and RX" (at 87.63 43.18 0) (fields_autoplaced)
-    (effects (font (size 5 5)) (justify left bottom))
   )
   (global_label "USB_CONNECTED" (shape input) (at 154.94 66.04 0) (fields_autoplaced)

Commit message: Bord v1.2, added flash memory, changed pinout od servomotor connectors and removed potentiometer signal from servomotors plus one ADC
Parts:
- removed SW1: SW_DIP_x01, Button_Switch_THT:SW_PUSH-12mm, symbol Switch:SW_DIP_x01
- renumbered U1 to U501
Connections:
- net FLASH_WP: now reaches U501.31 (GPIO26_ADC0)
- net FLASH_HOLD: now reaches U501.32 (GPIO27_ADC1)
Changed lines of the file:
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@@
 (kicad_sch (version 20230121) (generator eeschema)
   (paper "A4")
-  (junction (at 190.5 96.52) (diameter 0) (color 0 0 0 0)
-  )
   (wire (pts (xy 115.57 111.76) (xy 119.38 111.76))
     (stroke (width 0) (type default))
@@
     (stroke (width 0) (type default))
   )
-  (wire (pts (xy 190.5 91.44) (xy 190.5 96.52))
-    (stroke (width 0) (type default))
-  )
   (wire (pts (xy 161.29 93.98) (xy 154.94 93.98))
     (stroke (width 0) (type default))
@@
     (stroke (width 0) (type default))
   )
-  (wire (pts (xy 154.94 83.82) (xy 172.72 83.82))
-    (stroke (width 0) (type default))
-  )
-  (wire (pts (xy 175.26 91.44) (xy 154.94 91.44))
+  (wire (pts (xy 190.5 85.09) (xy 190.5 83.82))
     (stroke (width 0) (type default))
   )
@@
     (stroke (width 0) (type default))
   )
+  (wire (pts (xy 190.5 83.82) (xy 154.94 83.82))
+    (stroke (width 0) (type default))
+  )
   (wire (pts (xy 115.57 101.6) (xy 119.38 101.6))
     (stroke (width 0) (type default))
@@
   )
   (bus (pts (xy 154.94 101.6) (xy 161.29 101.6))
+    (stroke (width 0) (type default))
+  )
+  (wire (pts (xy 154.94 86.36) (xy 161.29 86.36))
+    (stroke (width 0) (type default))
+  )
+  (wire (pts (xy 154.94 88.9) (xy 161.29 88.9))
     (stroke (width 0) (type default))
   )
@@
     (effects (font (size 1.27 1.27)) (justify left))
   )
+  (hierarchical_label "FLASH_HOLD" (shape output) (at 161.29 86.36 0) (fields_autoplaced)
+    (effects (font (size 1.27 1.27)) (justify left))
+  )
   (hierarchical_label "I2C_SCL" (shape output) (at 161.29 99.06 0) (fields_autoplaced)
+    (effects (font (size 1.27 1.27)) (justify left))
+  )
+  (hierarchical_label "FLASH_WP" (shape output) (at 161.29 88.9 0) (fields_autoplaced)
     (effects (font (size 1.27 1.27)) (justify left))
   )
@@
     (effects (font (size 1.27 1.27)) (justify right))
   )
-  (symbol (lib_id "Switch:SW_DIP_x01") (at 182.88 91.44 0) (unit 1)
-    (in_bom yes) (on_board yes) (dnp no) (fields_autoplaced)
-    (property "Reference" "SW1" (at 182.88 83.82 0)
-      (effects (font (size 1.27 1.27)))
-    )
-    (property "Value" "SW_DIP_x01" (at 182.88 86.36 0)
-      (effects (font (size 1.27 1.27)))
-    )
-    (property "Footprint" "Button_Switch_THT:SW_PUSH-12mm" (at 182.88 91.44 0)
-      (effects (font (size 1.27 1.27)) hide)
-    )
-    (property "Datasheet" "~" (at 182.88 91.44 0)
-      (effects (font (size 1.27 1.27)) hide)
-    )
-    (pin "1")
-    (pin "2")
-    (instances
-      (project "Hexapod_Hardware"
-        (path "/04005f68-61ba-4735-aba3-9cac296c0cce/a539e409-d551-46bc-9b5e-4b2b4775713e"
-          (reference "SW1") (unit 1)
-        )
-      )
-    )
-  )
   (symbol (lib_id "power:GND") (at 190.5 109.22 0) (unit 1)
     (in_bom yes) (on_board yes) (dnp no)
-    (property "Reference" "#PWR036" (at 190.5 115.57 0)
+    (property "Reference" "#PWR0511" (at 190.5 115.57 0)
       (effects (font (size 1.27 1.27)) hide)
     )
@@
       (project "Hexapod_Hardware"
         (path "/04005f68-61ba-4735-aba3-9cac296c0cce/a539e409-d551-46bc-9b5e-4b2b4775713e"
-          (reference "#PWR036") (unit 1)
+          (reference "#PWR0511") (unit 1)
         )
       )
@@
   (symbol (lib_id "power:GND") (at 91.44 83.82 0) (unit 1)
     (in_bom yes) (on_board yes) (dnp no)
-    (property "Reference" "#PWR027" (at 91.44 90.17 0)
+    (property "Reference" "#PWR0502" (at 91.44 90.17 0)
       (effects (font (size 1.27 1.27)) hide)
     )
@@
       (project "Hexapod_Hardware"
         (path "/04005f68-61ba-4735-aba3-9cac296c0cce/a539e409-d551-46bc-9b5e-4b2b4775713e"
-          (reference "#PWR027") (unit 1)
+          (reference "#PWR0502") (unit 1)
         )
       )
@@
   (symbol (lib_id "power:GND") (at 91.44 71.12 0) (unit 1)
     (in_bom yes) (on_board yes) (dnp no)
-    (property "Reference" "#PWR026" (at 91.44 77.47 0)
+    (property "Reference" "#PWR0501" (at 91.44 77.47 0)
       (effects (font (size 1.27 1.27)) hide)
     )
@@
       (project "Hexapod_Hardware"
         (path "/04005f68-61ba-4735-aba3-9cac296c0cce/a539e409-d551-46bc-9b5e-4b2b4775713e"
-          (reference "#PWR026") (unit 1)
+          (reference "#PWR0501") (unit 1)
         )
       )
@@
   (symbol (lib_id "power:GND") (at 137.16 125.73 0) (unit 1)
     (in_bom yes) (on_board yes) (dnp no) (fields_autoplaced)
-    (property "Reference" "#PWR030" (at 137.16 132.08 0)
+    (property "Reference" "#PWR0505" (at 137.16 132.08 0)
       (effects (font (size 1.27 1.27)) hide)
     )
@@
       (project "Hexapod_Hardware"
         (path "/04005f68-61ba-4735-aba3-9cac296c0cce/a539e409-d551-46bc-9b5e-4b2b4775713e"
-          (reference "#PWR030") (unit 1)
+          (reference "#PWR0505") (unit 1)
         )
       )
@@
   (symbol (lib_id "power:GND") (at 190.5 96.52 0) (unit 1)
     (in_bom yes) (on_board yes) (dnp no)
-    (property "Reference" "#PWR035" (at 190.5 102.87 0)
+    (property "Reference" "#PWR0510" (at 190.5 102.87 0)
       (effects (font (size 1.27 1.27)) hide)
     )
@@
       (project "Hexapod_Hardware"
         (path "/04005f68-61ba-4735-aba3-9cac296c0cce/a539e409-d551-46bc-9b5e-4b2b4775713e"
-          (reference "#PWR035") (unit 1)
-        )
-      )
-    )
-  )
-  (symbol (lib_id "power:GND") (at 172.72 83.82 0) (unit 1)
-    (in_bom yes) (on_board yes) (dnp no)
-    (property "Reference" "#PWR032" (at 172.72 90.17 0)
-      (effects (font (size 1.27 1.27)) hide)
-    )
-    (property "Value" "GND" (at 172.72 87.63 0)
-      (effects (font (size 1.27 1.27)))
-    )
-    (property "Footprint" "" (at 172.72 83.82 0)
-      (effects (font (size 1.27 1.27)) hide)
-    )
-    (property "Datasheet" "" (at 172.72 83.82 0)
-      (effects (font (size 1.27 1.27)) hide)
-    )
-    (pin "1")
-    (instances
-      (project "Hexapod_Hardware"
-        (path "/04005f68-61ba-4735-aba3-9cac296c0cce/a539e409-d551-46bc-9b5e-4b2b4775713e"
-          (reference "#PWR032") (unit 1)
+          (reference "#PWR0510") (unit 1)
+        )
+      )
+    )
+  )
+  (symbol (lib_id "power:GND") (at 190.5 85.09 0) (unit 1)
+    (in_bom yes) (on_board yes) (dnp no)
+    (property "Reference" "#PWR0509" (at 190.5 91.44 0)
+      (effects (font (size 1.27 1.27)) hide)
+    )
+    (property "Value" "GND" (at 190.5 88.9 0)
+      (effects (font (size 1.27 1.27)))
+    )
+    (property "Footprint" "" (at 190.5 85.09 0)
+      (effects (font (size 1.27 1.27)) hide)
+    )
+    (property "Datasheet" "" (at 190.5 85.09 0)
+      (effects (font (size 1.27 1.27)) hide)
+    )
+    (pin "1")
+    (instances
+      (project "Hexapod_Hardware"
+        (path "/04005f68-61ba-4735-aba3-9cac296c0cce/a539e409-d551-46bc-9b5e-4b2b4775713e"
+          (reference "#PWR0509") (unit 1)
         )
       )
@@
   (symbol (lib_id "MCU_RaspberryPi_and_Boards:Pico") (at 137.16 90.17 0) (unit 1)
     (in_bom yes) (on_board yes) (dnp no) (fields_autoplaced)
-    (property "Reference" "U1" (at 137.16 59.69 0)
+    (property "Reference" "U501" (at 137.16 59.69 0)
       (effects (font (size 1.27 1.27)))
     )
@@
       (project "Hexapod_Hardware"
         (path "/04005f68-61ba-4735-aba3-9cac296c0cce/a539e409-d551-46bc-9b5e-4b2b4775713e"
-          (reference "U1") (unit 1)
+          (reference "U501") (unit 1)
         )
       )
@@
   (symbol (lib_id "power:+3.3V") (at 161.29 76.2 0) (unit 1)
     (in_bom yes) (on_board yes) (dnp no)
-    (property "Reference" "#PWR031" (at 161.29 80.01 0)
+    (property "Reference" "#PWR0506" (at 161.29 80.01 0)
       (effects (font (size 1.27 1.27)) hide)
     )
@@
       (project "Hexapod_Hardware"
         (path "/04005f68-61ba-4735-aba3-9cac296c0cce/a539e409-d551-46bc-9b5e-4b2b4775713e"
-          (reference "#PWR031") (unit 1)
+          (reference "#PWR0506") (unit 1)
         )
       )
@@
   (symbol (lib_id "power:+5V") (at 173.99 66.04 0) (unit 1)
     (in_bom yes) (on_board yes) (dnp no) (fields_autoplaced)
-    (property "Reference" "#PWR033" (at 173.99 69.85 0)
+    (property "Reference" "#PWR0507" (at 173.99 69.85 0)
       (effects (font (size 1.27 1.27)) hide)
     )
@@
       (project "Hexapod_Hardware"
         (path "/04005f68-61ba-4735-aba3-9cac296c0cce/a539e409-d551-46bc-9b5e-4b2b4775713e"
-          (reference "#PWR033") (unit 1)
+          (reference "#PWR0507") (unit 1)
         )
       )
@@
   (symbol (lib_id "power:GND") (at 173.99 71.12 0) (unit 1)
     (in_bom yes) (on_board yes) (dnp no) (fields_autoplaced)
-    (property "Reference" "#PWR034" (at 173.99 77.47 0)
+    (property "Reference" "#PWR0508" (at 173.99 77.47 0)
       (effects (font (size 1.27 1.27)) hide)
     )
@@
       (project "Hexapod_Hardware"
         (path "/04005f68-61ba-4735-aba3-9cac296c0cce/a539e409-d551-46bc-9b5e-4b2b4775713e"
-          (reference "#PWR034") (unit 1)
+          (reference "#PWR0508") (unit 1)
         )
       )
@@
   (symbol (lib_id "power:GND") (at 91.44 96.52 0) (unit 1)
     (in_bom yes) (on_board yes) (dnp no)
-    (property "Reference" "#PWR028" (at 91.44 102.87 0)
+    (property "Reference" "#PWR0503" (at 91.44 102.87 0)
       (effects (font (size 1.27 1.27)) hide)
     )
@@
       (project "Hexapod_Hardware"
         (path "/04005f68-61ba-4735-aba3-9cac296c0cce/a539e409-d551-46bc-9b5e-4b2b4775713e"
-          (reference "#PWR028") (unit 1)
+          (reference "#PWR0503") (unit 1)
         )
       )
@@
   (symbol (lib_id "power:GND") (at 91.44 109.22 0) (unit 1)
     (in_bom yes) (on_board yes) (dnp no)
-    (property "Reference" "#PWR029" (at 91.44 115.57 0)
+    (property "Reference" "#PWR0504" (at 91.44 115.57 0)
       (effects (font (size 1.27 1.27)) hide)
     )
@@
       (project "Hexapod_Hardware"
         (path "/04005f68-61ba-4735-aba3-9cac296c0cce/a539e409-d551-46bc-9b5e-4b2b4775713e"
-          (reference "#PWR029") (unit 1)
-        )
-      )
+          (reference "#PWR0504") (unit 1)
+        )
+      )
