File: adc.kicad_sch (KiCad schematic)
At the start: 0 parts

Commit message: cleaning up
Other:
- sheet ADC: file untitled.kicad_sch -> adc_converters.kicad_sch
Changed lines of the file:
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@@
       (effects (font (size 1.27 1.27)) (justify left bottom))
     )
-    (property "Sheetfile" "untitled.kicad_sch" (at 161.29 155.5246 0)
+    (property "Sheetfile" "adc_converters.kicad_sch" (at 161.29 155.5246 0)
       (effects (font (size 1.27 1.27)) (justify left top))
     )

Commit message: Bord v1.2, added flash memory, changed pinout od servomotor connectors and removed potentiometer signal from servomotors plus one ADC
Other:
- sheet ADC ports: added none; removed SPI_CS_2
Changed lines of the file:
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@@
-    (stroke (width 0) (type default))
-  )
-  (bus (pts (xy 201.93 109.22) (xy 210.82 109.22))
     (stroke (width 0) (type default))
   )
@@
   (hierarchical_label "SERVO_PWM_1" (shape input) (at 102.87 49.53 180) (fields_autoplaced)
     (effects (font (size 1.27 1.27)) (justify right))
-  )
-  (hierarchical_label "SPI_CS_2" (shape input) (at 210.82 109.22 0) (fields_autoplaced)
-    (effects (font (size 1.27 1.27)) (justify left))
   )
   (hierarchical_label "SPI_CS_0" (shape input) (at 210.82 104.14 0) (fields_autoplaced)
@@
       (effects (font (size 1.27 1.27)) (justify right))
     )
-    (pin "SPI_CS_2" input (at 201.93 109.22 0)
-      (effects (font (size 1.27 1.27)) (justify right))
-    )
