File: gripper.kicad_sch (KiCad schematic)
At the start: 1 part, among them J23 Conn_01x03

Commit message: Bord v1.2, added flash memory, changed pinout od servomotor connectors and removed potentiometer signal from servomotors plus one ADC
Parts:
- renumbered J23 to J201
Connections:
- net MCU_GRIPPER/SWCLK: now also J201.2 (Pin_2); no longer J201.1 (Pin_1)
- net MCU_GRIPPER/SWDIO: now also J201.1 (Pin_1); no longer J201.2 (Pin_2)
Changed lines of the file:
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@@
+    (stroke (width 0) (type default))
+  )
+  (wire (pts (xy 163.83 100.33) (xy 166.37 100.33))
+    (stroke (width 0) (type default))
+  )
+  (wire (pts (xy 163.83 113.03) (xy 171.45 113.03))
+    (stroke (width 0) (type default))
+  )
+  (wire (pts (xy 109.22 109.22) (xy 116.84 109.22))
+    (stroke (width 0) (type default))
+  )
+  (wire (pts (xy 109.22 144.78) (xy 116.84 144.78))
+    (stroke (width 0) (type default))
+  )
+  (wire (pts (xy 163.83 105.41) (xy 166.37 105.41))
+    (stroke (width 0) (type default))
+  )
+  (wire (pts (xy 109.22 123.19) (xy 116.84 123.19))
+    (stroke (width 0) (type default))
+  )
+  (wire (pts (xy 109.22 137.16) (xy 116.84 137.16))
+    (stroke (width 0) (type default))
+  )
+  (wire (pts (xy 109.22 106.68) (xy 116.84 106.68))
+    (stroke (width 0) (type default))
+  )
+  (wire (pts (xy 109.22 104.14) (xy 116.84 104.14))
+    (stroke (width 0) (type default))
+  )
+  (wire (pts (xy 163.83 132.08) (xy 171.45 132.08))
+    (stroke (width 0) (type default))
+  )
+  (wire (pts (xy 109.22 120.65) (xy 116.84 120.65))
     (stroke (width 0) (type default))
   )
@@
     (stroke (width 0) (type default))
   )
-  (wire (pts (xy 163.83 113.03) (xy 171.45 113.03))
-    (stroke (width 0) (type default))
-  )
-  (wire (pts (xy 109.22 109.22) (xy 116.84 109.22))
-    (stroke (width 0) (type default))
-  )
-  (wire (pts (xy 109.22 144.78) (xy 116.84 144.78))
-    (stroke (width 0) (type default))
-  )
-  (wire (pts (xy 163.83 105.41) (xy 166.37 105.41))
-    (stroke (width 0) (type default))
-  )
-  (wire (pts (xy 109.22 123.19) (xy 116.84 123.19))
-    (stroke (width 0) (type default))
-  )
-  (wire (pts (xy 109.22 137.16) (xy 116.84 137.16))
-    (stroke (width 0) (type default))
-  )
-  (wire (pts (xy 109.22 106.68) (xy 116.84 106.68))
-    (stroke (width 0) (type default))
-  )
-  (wire (pts (xy 109.22 104.14) (xy 116.84 104.14))
-    (stroke (width 0) (type default))
-  )
-  (wire (pts (xy 163.83 132.08) (xy 171.45 132.08))
-    (stroke (width 0) (type default))
-  )
-  (wire (pts (xy 109.22 120.65) (xy 116.84 120.65))
-    (stroke (width 0) (type default))
-  )
   (wire (pts (xy 109.22 139.7) (xy 116.84 139.7))
     (stroke (width 0) (type default))
@@
   )
   (wire (pts (xy 163.83 124.46) (xy 171.45 124.46))
-    (stroke (width 0) (type default))
-  )
-  (wire (pts (xy 163.83 100.33) (xy 166.37 100.33))
     (stroke (width 0) (type default))
   )
@@
   (symbol (lib_id "Connector_Generic:Conn_01x03") (at 171.45 102.87 0) (unit 1)
     (in_bom yes) (on_board yes) (dnp no) (fields_autoplaced)
-    (property "Reference" "J23" (at 173.99 102.235 0)
+    (property "Reference" "J201" (at 173.99 102.235 0)
       (effects (font (size 1.27 1.27)) (justify left))
     )
@@
     (instances
       (project "Hexapod_Hardware"
-        (path "/04005f68-61ba-4735-aba3-9cac296c0cce/131ce24a-6b68-4bf4-9124-91468713a7c9"
-          (reference "J23") (unit 1)
+        (path "/04005f68-61ba-4735-aba3-9cac296c0cce/2cd4ba25-52d1-4db4-b74d-e04810e070ce/59004b94-8694-4dc2-864b-96bb314c80e0"
+          (reference "J201") (unit 1)
         )
       )
@@
   (symbol (lib_id "power:+6V") (at 86.36 85.09 0) (unit 1)
     (in_bom yes) (on_board yes) (dnp no) (fields_autoplaced)
-    (property "Reference" "#PWR071" (at 86.36 88.9 0)
+    (property "Reference" "#PWR0201" (at 86.36 88.9 0)
       (effects (font (size 1.27 1.27)) hide)
     )
@@
     (instances
       (project "Hexapod_Hardware"
-        (path "/04005f68-61ba-4735-aba3-9cac296c0cce/131ce24a-6b68-4bf4-9124-91468713a7c9"
-          (reference "#PWR071") (unit 1)
+        (path "/04005f68-61ba-4735-aba3-9cac296c0cce/2cd4ba25-52d1-4db4-b74d-e04810e070ce/59004b94-8694-4dc2-864b-96bb314c80e0"
+          (reference "#PWR0201") (unit 1)
         )
       )
@@
     (instances
       (project "Hexapod_Hardware"
-        (path "/04005f68-61ba-4735-aba3-9cac296c0cce/131ce24a-6b68-4bf4-9124-91468713a7c9" (page "11"))
+        (path "/04005f68-61ba-4735-aba3-9cac296c0cce/2cd4ba25-52d1-4db4-b74d-e04810e070ce/59004b94-8694-4dc2-864b-96bb314c80e0" (page "9"))
       )
     )
@@
       (effects (font (size 1.27 1.27)) (justify left))
     )
-    (pin "SWDIO" bidirectional (at 163.83 102.87 0)
+    (pin "SWDIO" bidirectional (at 163.83 100.33 0)
       (effects (font (size 1.27 1.27)) (justify right))
     )
@@
       (effects (font (size 1.27 1.27)) (justify right))
     )
-    (pin "SWCLK" input (at 163.83 100.33 0)
+    (pin "SWCLK" input (at 163.83 102.87 0)
       (effects (font (size 1.27 1.27)) (justify right))
     )
@@
     (instances
       (project "Hexapod_Hardware"
-        (path "/04005f68-61ba-4735-aba3-9cac296c0cce/131ce24a-6b68-4bf4-9124-91468713a7c9" (page "11"))
-      )
-    )
+        (path "/04005f68-61ba-4735-aba3-9cac296c0cce/2cd4ba25-52d1-4db4-b74d-e04810e070ce/59004b94-8694-4dc2-864b-96bb314c80e0" (page "6"))
+      )
+    )
