File: test_ADC_and_CurrentSensors/test_ADC_and_CurrentSensors.kicad_sch (KiCad schematic)
At the start: 25 parts, among them IC1 MCS1802GS-05-Z, IC2 STM32G030K8T6, IC3 MCP3008-I_SL, J1 Conn_01x04_Male, J2 Conn_01x05_Female, J3 Conn_01x03_Female, J4 Conn_01x06_Female, J5 Conn_01x02_Pin, J9 Conn_01x02_Pin, U1 LM2902

Commit message: cleaning up
Parts:
- R10, R9: value R -> 47k
- R3, R7, R8: value R -> 10k
- R4: value R -> 6k8
- R5: value R -> 1k
- R6: value R -> 2k
Other:
- sheet LDO: file untitled.kicad_sch -> Voltage_regulators.kicad_sch
- note removed: "CHECK SERVO POTENTIOMETER VOLTAGES!"
- moved on the sheet: R4
Changed lines of the file:
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@@
+    (stroke (width 0) (type default))
+  )
+  (wire (pts (xy 77.47 124.46) (xy 77.47 123.19))
     (stroke (width 0) (type default))
   )
@@
   )
   (text "TO CONSIDER:\n-> MORE SERVOMOTORS\n-> CHECK MCU ELECTRO\n-> LOW DROPDOWN REGULATOR (LDO)\n "
-    (at 156.21 100.33 0)
+    (at 157.48 99.06 0)
     (effects (font (size 1.27 1.27) italic) (justify left bottom))
-  )
-  (text "CHECK SERVO POTENTIOMETER VOLTAGES!" (at 68.58 8.89 0)
-    (effects (font (size 5 5)) (justify left bottom))
   )
   (text "SPI COMMUNICATION" (at 113.03 55.88 0)
@@
   (symbol (lib_id "Device:R") (at 110.49 120.65 0) (unit 1)
     (in_bom yes) (on_board yes) (dnp no) (fields_autoplaced)
-    (property "Reference" "R9" (at 113.03 119.3799 0)
-      (effects (font (size 1.27 1.27)) (justify left))
-    )
-    (property "Value" "R" (at 113.03 121.9199 0)
+    (property "Reference" "R9" (at 113.03 120.015 0)
+      (effects (font (size 1.27 1.27)) (justify left))
+    )
+    (property "Value" "47k" (at 113.03 122.555 0)
       (effects (font (size 1.27 1.27)) (justify left))
     )
@@
   (symbol (lib_id "Device:R") (at 85.09 181.61 0) (unit 1)
     (in_bom yes) (on_board yes) (dnp no)
-    (property "Reference" "R6" (at 87.122 181.61 90)
-      (effects (font (size 1.27 1.27)))
-    )
-    (property "Value" "R" (at 85.09 181.61 90)
+    (property "Reference" "R6" (at 87.63 180.34 0)
+      (effects (font (size 1.27 1.27)))
+    )
+    (property "Value" "2k" (at 87.63 182.372 0)
       (effects (font (size 1.27 1.27)))
     )
@@
   (symbol (lib_id "Device:R") (at 77.47 118.11 0) (unit 1)
     (in_bom yes) (on_board yes) (dnp no) (fields_autoplaced)
-    (property "Reference" "R3" (at 80.01 116.8399 0)
-      (effects (font (size 1.27 1.27)) (justify left))
-    )
-    (property "Value" "R" (at 80.01 119.3799 0)
+    (property "Reference" "R3" (at 80.01 117.475 0)
+      (effects (font (size 1.27 1.27)) (justify left))
+    )
+    (property "Value" "10k" (at 80.01 120.015 0)
       (effects (font (size 1.27 1.27)) (justify left))
     )
@@
     )
   )
-  (symbol (lib_id "Device:R") (at 77.47 127 0) (unit 1)
+  (symbol (lib_id "Device:R") (at 77.47 128.27 0) (unit 1)
     (in_bom yes) (on_board yes) (dnp no)
-    (property "Reference" "R4" (at 79.502 127 90)
-      (effects (font (size 1.27 1.27)))
-    )
-    (property "Value" "R" (at 77.47 127 90)
-      (effects (font (size 1.27 1.27)))
-    )
-    (property "Footprint" "Resistor_SMD:R_1206_3216Metric" (at 75.692 127 90)
-      (effects (font (size 1.27 1.27)) hide)
-    )
-    (property "Datasheet" "~" (at 77.47 127 0)
+    (property "Reference" "R4" (at 81.28 129.54 0)
+      (effects (font (size 1.27 1.27)))
+    )
+    (property "Value" "6k8" (at 81.28 127 0)
+      (effects (font (size 1.27 1.27)))
+    )
+    (property "Footprint" "Resistor_SMD:R_1206_3216Metric" (at 75.692 128.27 90)
+      (effects (font (size 1.27 1.27)) hide)
+    )
+    (property "Datasheet" "~" (at 77.47 128.27 0)
       (effects (font (size 1.27 1.27)) hide)
     )
@@
     )
   )
-  (symbol (lib_id "power:GND") (at 77.47 130.81 0) (unit 1)
-    (in_bom yes) (on_board yes) (dnp no) (fields_autoplaced)
-    (property "Reference" "#PWR09" (at 77.47 137.16 0)
-      (effects (font (size 1.27 1.27)) hide)
-    )
-    (property "Value" "GND" (at 77.47 135.89 0)
-      (effects (font (size 1.27 1.27)))
-    )
-    (property "Footprint" "" (at 77.47 130.81 0)
-      (effects (font (size 1.27 1.27)) hide)
-    )
-    (property "Datasheet" "" (at 77.47 130.81 0)
+  (symbol (lib_id "power:GND") (at 77.47 132.08 0) (unit 1)
+    (in_bom yes) (on_board yes) (dnp no) (fields_autoplaced)
+    (property "Reference" "#PWR09" (at 77.47 138.43 0)
+      (effects (font (size 1.27 1.27)) hide)
+    )
+    (property "Value" "GND" (at 77.47 137.16 0)
+      (effects (font (size 1.27 1.27)))
+    )
+    (property "Footprint" "" (at 77.47 132.08 0)
+      (effects (font (size 1.27 1.27)) hide)
+    )
+    (property "Datasheet" "" (at 77.47 132.08 0)
       (effects (font (size 1.27 1.27)) hide)
     )
@@
       (effects (font (size 1.27 1.27)))
     )
-    (property "Value" "R" (at 129.54 97.79 90)
+    (property "Value" "47k" (at 129.54 97.79 90)
       (effects (font (size 1.27 1.27)))
     )
@@
       (effects (font (size 1.27 1.27)))
     )
-    (property "Value" "R" (at 102.87 110.49 90)
+    (property "Value" "10k" (at 102.87 110.49 90)
       (effects (font (size 1.27 1.27)))
     )
@@
       (effects (font (size 1.27 1.27)))
     )
-    (property "Value" "R" (at 104.14 97.79 90)
+    (property "Value" "10k" (at 104.14 97.79 90)
       (effects (font (size 1.27 1.27)))
     )
@@
   )
   (symbol (lib_id "Device:R") (at 85.09 172.72 0) (unit 1)
-    (in_bom yes) (on_board yes) (dnp no) (fields_autoplaced)
-    (property "Reference" "R5" (at 87.63 171.4499 0)
-      (effects (font (size 1.27 1.27)) (justify left))
-    )
-    (property "Value" "R" (at 87.63 173.9899 0)
+    (in_bom yes) (on_board yes) (dnp no)
+    (property "Reference" "R5" (at 86.36 171.45 0)
+      (effects (font (size 1.27 1.27)) (justify left))
+    )
+    (property "Value" "1k" (at 86.36 173.99 0)
       (effects (font (size 1.27 1.27)) (justify left))
     )
@@
       (effects (font (size 1.27 1.27)) (justify left bottom))
     )
-    (property "Sheetfile" "untitled.kicad_sch" (at 162.56 39.9546 0)
+    (property "Sheetfile" "Voltage_regulators.kicad_sch" (at 162.56 39.9546 0)
       (effects (font (size 1.27 1.27)) (justify left top))
     )

Commit message: ordered pcbs
Parts:
- R10, R9: value 47k -> 100k
Changed lines of the file:
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@@
       (effects (font (size 1.27 1.27)) (justify left))
     )
-    (property "Value" "47k" (at 113.03 122.555 0)
+    (property "Value" "100k" (at 113.03 122.555 0)
       (effects (font (size 1.27 1.27)) (justify left))
     )
@@
       (effects (font (size 1.27 1.27)))
     )
-    (property "Value" "47k" (at 129.54 97.79 90)
-      (effects (font (size 1.27 1.27)))
-    )
+    (property "Value" "100k" (at 129.54 97.79 90)
+      (effects (font (size 1.27 1.27)))
+    )

Commit message: new pcb
Parts:
- R1: value R -> 0.180R
Changed lines of the file:
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@@
   (symbol (lib_id "Device:R") (at 43.18 104.14 0) (unit 1)
     (in_bom yes) (on_board yes) (dnp no) (fields_autoplaced)
-    (property "Reference" "R1" (at 45.72 102.8699 0)
+    (property "Reference" "R1" (at 45.72 103.505 0)
       (effects (font (size 1.27 1.27)) (justify left))
     )
-    (property "Value" "R" (at 45.72 105.4099 0)
+    (property "Value" "0.180R" (at 45.72 106.045 0)
       (effects (font (size 1.27 1.27)) (justify left))
     )
